Commit message: femur mesh

File: src/model/urdf/pidog.urdf (robot description, URDF)
Before this commit: robot pidog, 3 links, 2 joints
Links:
- link left_back_leg: geometry visual mesh filename=package://model/meshes/femur.dae
- link left_front_leg: geometry visual mesh filename=package://model/meshes/femur.dae

Commit message: dae file is sized massively, needs to be scaled way down

File: src/model/urdf/pidog.urdf (robot description, URDF)
Before this commit: robot pidog, 6 links, 5 joints
Links:
- link left_front_leg: geometry visual mesh filename=package://model/meshes/l_finger.dae

Commit message: left legs seemingly attached correctly but right legs need work

File: src/model/urdf/pidog.urdf (robot description, URDF)
Before this commit: robot pidog, 6 links, 5 joints
Links:
- link left_front_leg: geometry visual mesh filename=package://model/meshes/femur.dae

Commit message: 0 out the right front leg

File: src/model/urdf/pidog.urdf (robot description, URDF)
Before this commit: robot pidog, 4 links, 3 joints
Joints:
- joint body_to_right_front_leg: origin xyz=0.092 -0.082 0 rpy=0 -0.8 0 -> xyz=0 0 0 rpy=0 0 0

Commit message: add in the front right tibia

File: src/model/urdf/pidog.urdf (robot description, URDF)
Before this commit: robot pidog, 5 links, 4 joints
Links:
- removed link right_front_leg
- added link right_front_femur; visual mesh filename=package://model/meshes/femur.dae
- added link right_front_tibia; visual mesh filename=package://model/meshes/tibia_R.dae
Joints:
- removed joint body_to_right_front_leg
- added joint body_to_right_front_femur: type fixed, parent base_link, child right_front_femur, origin xyz=0.092 -0.082 0 rpy=0 1 0
- added joint right_front_femur_to_tibia: type fixed, parent right_front_femur, child fright_front_tibia, origin xyz=0 0 0 rpy=0 0 0

Commit message: clean

File: src/model/urdf/pidog.urdf (robot description, URDF)
Before this commit: robot pidog, 6 links, 5 joints
Links:
- removed link right_front_tibia
Joints:
- removed joint right_front_femur_to_tibia

Commit message: tibia

File: src/model/urdf/pidog.urdf (robot description, URDF)
Before this commit: robot pidog, 5 links, 4 joints
Links:
- added link right_front_tibia; visual mesh filename=package://model/meshes/tibia_R.dae
Joints:
- added joint right_front_femur_to_tibia: type fixed, parent right_front_femur, child fright_front_tibia, origin xyz=0 0 0 rpy=0 0 0

Commit message: typo

File: src/model/urdf/pidog.urdf (robot description, URDF)
Before this commit: robot pidog, 6 links, 5 joints
Joints:
- joint right_front_femur_to_tibia: child fright_front_tibia -> right_front_tibia

Commit message: full robot dae

File: src/model/urdf/pidog.urdf (robot description, URDF)
Before this commit: robot pidog, 6 links, 5 joints
Joints:
- joint body_to_right_front_femur: axis (none) -> 0 0 -1; limit (none) -> lower=0.0 upper=0.548 effort=1000.0 velocity=0.5; type fixed -> revolute
