Commit message: sized base_link

File: src/model/urdf/quadruped.xacro (robot description, xacro)
@@ -1,4 +1,10 @@
 <?xml version="1.0"?>
 <robot xmlns:xacro="http://www.ros.org/wiki/xacro" name="pidog">
+  <material name="white">
+    <color rgba="1 1 1 1" />
+  </material>
+  <material name="red">
+    <color rgba="1 0 0 1" />
+  </material>
   <xacro:property name="bodylength" value="0.3048" />
   <xacro:property name="bodywidth" value="0.127" />
@@ -7,5 +13,4 @@
   <xacro:property name="femurwidth" value="0.12065" />
   <xacro:macro name="femur" params="prefix reflect">
-    <!-- This is only an example. This needs to be updated to correctly represent the quadruped -->
     <link name="${prefix}_femur">
         <visual>
@@ -13,5 +18,5 @@
                 <box size="${femurlength} 0.1 0.2"/>
             </geometry>
-            <origin xyz="0 0 -${femurlength/2}" rpy="0 ${pi/2} 0"/>
+            <origin xyz="0 0 0" rpy="0 0 0"/>
             <material name="white"/>
         </visual>
@@ -20,5 +25,5 @@
                 <box size="${femurlength} 0.1 0.2"/>
             </geometry>
-            <origin xyz="0 0 -${femurlength/2}" rpy="0 ${pi/2} 0"/>
+            <origin xyz="0 0 0" rpy="0 0 0"/>
         </collision>
         <xacro:default_inertial mass="10"/>
@@ -36,17 +41,15 @@
         <box size="${bodylength} ${bodywidth} ${bodyheight}" />
       </geometry>
-      <material name="gray">
-        <color rgba=".2 .2 .2 1" />
-      </material>
+      <material name="red"/>
     </visual>
     <collision>
-      <origin xyz="0 0 0" rpy="1.57 0 0" />
+      <origin xyz="0 0 0" rpy="0 0 0" />
       <geometry>
-        <box size="0.3048 0.127 0.762" />
+        <box size="${bodylength} ${bodywidth} ${bodyheight}" />
       </geometry>
       <contact_coefficients mu="0" kp="1000.0" kd="1.0"/>
     </collision>
   </link>
-  <xacro:leg prefix="right" reflect="1" />
-  <xacro:leg prefix="left" reflect="-1" />
+  <xacro:femur prefix="front_right" reflect="1" />
+  <!-- <xacro:femur prefix="left" reflect="-1" /> -->
 </robot>

Commit message: add femur

File: src/model/urdf/quadruped.xacro (robot description, xacro)
@@ -14,23 +14,23 @@
   <xacro:macro name="femur" params="prefix reflect">
     <link name="${prefix}_femur">
-        <visual>
-            <geometry>
-                <box size="${femurlength} 0.1 0.2"/>
-            </geometry>
-            <origin xyz="0 0 0" rpy="0 0 0"/>
-            <material name="white"/>
-        </visual>
-        <collision>
-            <geometry>
-                <box size="${femurlength} 0.1 0.2"/>
-            </geometry>
-            <origin xyz="0 0 0" rpy="0 0 0"/>
-        </collision>
-        <xacro:default_inertial mass="10"/>
+      <visual>
+        <geometry>
+          <box size="${femurlength} 0.1 0.2"/>
+        </geometry>
+        <origin xyz="0 0 0" rpy="0 0 0"/>
+        <material name="white"/>
+      </visual>
+      <collision>
+        <geometry>
+          <box size="${femurlength} 0.1 0.2"/>
+        </geometry>
+        <origin xyz="0 0 0" rpy="0 0 0"/>
+      </collision>
+      <xacro:default_inertial mass="10"/>
     </link>
     <joint name="base_to_${prefix}_femur" type="fixed">
-        <parent link="base_link"/>
-        <child link="${prefix}_femur"/>
-        <origin xyz="0 ${reflect*(width+.02)} 0.25" />
+      <parent link="base_link"/>
+      <child link="${prefix}_femur"/>
+      <origin xyz="0 ${reflect*(width+.02)} 0.25" />
     </joint>
   </xacro:macro>
