Commit message: sync

File: install/model/share/model/urdf/pidog.urdf (robot description, URDF)
Before this commit: robot pidog, 3 links, 2 joints
Links:
- removed link body
- added link base_link; visual box size=0.28575 0.1397 0.05588
Joints:
- joint body_to_left_back_leg: parent body -> base_link
- joint body_to_left_front_leg: parent body -> base_link

Commit message: dae file is sized massively, needs to be scaled way down

File: install/model/share/model/urdf/pidog.urdf (robot description, URDF)
Before this commit: robot pidog, 3 links, 2 joints
Links:
- link left_back_leg: geometry visual mesh filename=package://model/meshes/femur.dae
- link left_front_leg: geometry visual mesh filename=package://model/meshes/l_finger.dae

File: src/model/urdf/pidog.urdf (robot description, URDF)
Before this commit: robot pidog, 3 links, 2 joints
Links:
- link left_front_leg: geometry visual mesh filename=package://model/meshes/l_finger.dae

Commit message: left legs seemingly attached correctly but right legs need work

File: install/model/share/model/urdf/pidog.urdf (robot description, URDF)
Before this commit: robot pidog, 3 links, 2 joints
Links:
- added link right_front_leg; visual mesh filename=package://model/meshes/femur.dae
- link left_front_leg: geometry visual mesh filename=package://model/meshes/femur.dae
Joints:
- added joint body_to_right_front_leg: type fixed, parent base_link, child right_front_leg, origin xyz=0.092 -0.082 0 rpy=0 -0.8 0
- joint body_to_left_back_leg: origin xyz=-0.092 0.082 0 -> xyz=-0.092 0.082 0 rpy=0 1.8 0
- joint body_to_left_front_leg: origin xyz=0.092 0.082 0 -> xyz=0.092 0.082 0 rpy=0 1.8 0

Commit message: front right is close

File: install/model/share/model/urdf/pidog.urdf (robot description, URDF)
Before this commit: robot pidog, 4 links, 3 joints
Joints:
- joint body_to_right_front_leg: origin xyz=0.092 -0.082 0 rpy=0 -0.8 0 -> xyz=0.092 -0.082 0 rpy=0 -1.5 0

File: src/model/urdf/pidog.urdf (robot description, URDF)
Before this commit: robot pidog, 4 links, 3 joints
Joints:
- joint body_to_right_front_leg: origin xyz=0 0 0 rpy=0 0 0 -> xyz=0.092 -0.082 0 rpy=0 -1.5 0

Commit message: femurs in place

File: install/model/share/model/urdf/pidog.urdf (robot description, URDF)
Before this commit: robot pidog, 4 links, 3 joints
Links:
- added link right_back_leg; visual mesh filename=package://model/meshes/femur.dae
Joints:
- added joint body_to_right_back_leg: type fixed, parent base_link, child right_back_leg, origin xyz=-0.092 -0.082 0 rpy=0 1 0
- joint body_to_right_front_leg: origin xyz=0.092 -0.082 0 rpy=0 -1.5 0 -> xyz=0.092 -0.082 0 rpy=0 1 0

Commit message: tibia is almost perfect

File: install/model/share/model/urdf/pidog.urdf (robot description, URDF)
Before this commit: robot pidog, 5 links, 4 joints
Links:
- removed link right_front_leg
- added link right_front_femur; visual mesh filename=package://model/meshes/femur.dae
- added link right_front_tibia; visual mesh filename=package://model/meshes/tibia_R.dae
Joints:
- removed joint body_to_right_front_leg
- added joint body_to_right_front_femur: type fixed, parent base_link, child right_front_femur, origin xyz=0.092 -0.082 0 rpy=0 1 0
- added joint right_front_femur_to_tibia: type fixed, parent right_front_femur, child right_front_tibia, origin xyz=0 0 -0.1 rpy=0 0 0

File: src/model/urdf/pidog.urdf (robot description, URDF)
Before this commit: robot pidog, 6 links, 5 joints
Joints:
- joint right_front_femur_to_tibia: origin xyz=0 0 0 rpy=0 0 0 -> xyz=0 0 -0.1 rpy=0 0 0
