Commit message: remove lower leg

File: src/urdf_tutorial_r2d2/urdf/quadruped.urdf (robot description, URDF)
Before this commit: robot quadruped_robot, 4 links, 3 joints
Links:
- removed link leg1_lower_leg
- removed link leg2_link
Joints:
- removed joint base_to_leg2
- removed joint leg1_femur_to_lower_leg

Commit message: only base link

File: src/urdf_tutorial_r2d2/urdf/quadruped.urdf (robot description, URDF)
Before this commit: robot quadruped_robot, 2 links, 1 joints
Links:
- removed link leg1_femur
Joints:
- removed joint base_to_leg1_femur
